File: laos-board-rev3/laos-board.sch (KiCad schematic (older format))
At the start: 99 parts, among them IC1 KB847, IC2 KB847, J1 USB-A, J10 I2C, J11 MBED NXP, J12 JP, J13 ZEXT, J14 ANALOG, J15 JP, J16 JP_3, J17 POLOLU1201, J18 YAXIS, J19 JP, J2 CAN, J20 YEXT, J21 JP, J22 JP_3, J23 POLOLU1201, J24 XAXIS, J25 JP, J26 XEXT, J27 OUTPUT, J28 VSENSOR, J29 INPUT12, J3 USBPWR, J30 JP, J31 JP_3, J32 POLOLU1201, J33 EAXIS, J34 INPUT34, J35 JP, J36 EEXT, J37 OUTPUT12, J38 VCPU, J39 OUTPUT34, J4 MAGJACK, J40 JP, J41 O1_SRC, J42 O2_SRC, J43 CONN_4, J5 CONN_3, J6 JP, J7 JP_3, J8 POLOLU1201, J9 ZAXIS, Q1 TIP115, Q2 TIP115, U1 65HVD251, U2 SDCARD, U3 7805

Commit message: changes made in Arnhem, ready to go?
Parts:
- removed C2: 100nF, Pkg, symbol C
Changed lines of the file:
@@
-EESchema Schematic File Version 2  date Wed 30 May 2012 10:33:13 PM CEST
+EESchema Schematic File Version 2  date Sat 02 Jun 2012 02:34:44 PM CEST
 LIBS:laos_kicad_lib
 LIBS:power
@@
 Sheet 1 1
 Title "LAOS"
-Date ""
+Date "2 jun 2012"
 Rev "3"
 Comp "http://www.laoslaser.org"
@@
 Connection ~ 3250 8400
 Connection ~ 3250 9000
-Connection ~ 2175 1125
 Wire Wire Line
 	2175 825  2175 1175
-Wire Wire Line
-	1775 1125 1775 825
 Wire Wire Line
 	1850 2550 1850 2400
@@
 $EndComp
 $Comp
-L C C2
-U 1 1 4E0B1D28
-P 1975 1125
-F 0 "C2" H 2075 1075 60  0000 C CNB
-F 1 "100nF" H 1575 1125 60  0000 C CNN
-F 2 "Pkg" H 1975 900 30  0001 C CNN
-	1    1975 1125
-	-1   0    0    1
-$EndComp
-$Comp

Commit message: added flatcable connector
Parts:
- added P1: FLATCONN, symbol CONN_12
Connections:
- net GND: now also P1.7 (P7)
- net at IC1.1, IC1.3 (A), IC1.5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: now also P1.10 (P10)
- net at J34.2 (P2), R26.2: now also P1.8 (P8)
- net at J34.3 (P3), R27.2: now also P1.9 (P9)
- net at J21.2, J23.14 (2B), J24.1 (P1): now also P1.1 (P1)
- net at J23.11 (1B), J24.4 (P4), J26.2 (P6): now also P1.4 (P4)
- net at J23.12 (1A), J24.3 (P3), J26.4 (P5): now also P1.3 (P3)
- net at J23.13 (2A), J24.2 (P2), J26.6 (P4): now also P1.2 (P2)
- no-connect marks 5 -> 9
